File: cantact.sch (KiCad schematic (older format))
At the start: 37 parts, among them P1 USB, P2 SWD, P3 DB9, U1 STM32F042C6T6, U2 AAT3221, U3 MCP2551-I/SN, X1 16 MHz

Commit message: read in the old schematic and reconnect all the changed symbols
Parts:
- removed P1: USB, Connect:USB_B, symbol USB
- removed TP1, TP2, TP3: TST, Connect:PINTST, symbol TST
- added P1: USB_B, symbol USB_B
- added TP1, TP2, TP3: TEST, symbol TEST
- X1: symbol CRYSTAL -> Crystal
Connections:
- wire segments 127 -> 134
- no-connect marks 0 -> 35
Other:
- moved on the sheet: R4
