File: cantransceiver.sch (KiCad schematic (older format))
At the start: 3 parts

Commit message: stuff
Parts:
- C36: renamed from C?; value 0.1uF -> 0.1u; footprint (none) -> Capacitors_SMD:C_0402; MPN (none) -> CL05B104KO5NNNC
- C37: renamed from C?; value 0.1uF -> 0.1u; footprint Capacitors_SMD:C_0603 -> Capacitors_SMD:C_0402
- gave numbers to parts that had none: 1
Changed lines of the file:
@@
 $EndDescr
 $Comp
-L GND #PWR?
+L GND #PWR066
 U 1 1 58D48959
 P 4000 3750
-F 0 "#PWR?" H 4000 3750 30  0001 C CNN
+F 0 "#PWR066" H 4000 3750 30  0001 C CNN
 F 1 "GND" H 4000 3680 30  0001 C CNN
 F 2 "" H 4000 3750 60  0000 C CNN
@@
 $EndComp
 $Comp
-L GND #PWR?
+L GND #PWR067
 U 1 1 58D4895F
 P 4550 3750
-F 0 "#PWR?" H 4550 3750 30  0001 C CNN
+F 0 "#PWR067" H 4550 3750 30  0001 C CNN
 F 1 "GND" H 4550 3680 30  0001 C CNN
 F 2 "" H 4550 3750 60  0000 C CNN
@@
 $EndComp
 $Comp
-L C C?
+L C C37
 U 1 1 58D48965
 P 4800 2750
-F 0 "C?" V 4850 2550 40  0000 L CNN
-F 1 "0.1uF" V 4900 2550 40  0000 L CNN
-F 2 "Capacitors_SMD:C_0603" H 4838 2600 30  0001 C CNN
+F 0 "C37" V 4850 2550 40  0000 L CNN
+F 1 "0.1u" V 4900 2550 40  0000 L CNN
+F 2 "Capacitors_SMD:C_0402" H 4838 2600 30  0001 C CNN
 F 3 "" H 4800 2750 60  0000 C CNN
 	1    4800 2750
@@
 $EndComp
 $Comp
-L GND #PWR?
+L GND #PWR068
 U 1 1 58D4896C
 P 5100 2900
-F 0 "#PWR?" H 5100 2900 30  0001 C CNN
+F 0 "#PWR068" H 5100 2900 30  0001 C CNN
 F 1 "GND" H 5100 2830 30  0001 C CNN
 F 2 "" H 5100 2900 60  0000 C CNN
@@
 $EndComp
 $Comp
-L +5V #PWR?
+L +5V #PWR069
 U 1 1 58D48972
 P 4550 2700
-F 0 "#PWR?" H 4550 2790 20  0001 C CNN
+F 0 "#PWR069" H 4550 2790 20  0001 C CNN
 F 1 "+5V" H 4550 2790 30  0000 C CNN
 F 2 "" H 4550 2700 60  0000 C CNN
@@
 $EndComp
 $Comp
-L MCP2562-E/SN U?
+L MCP2562-E/SN U4
 U 1 1 58D48980
 P 4550 3250
-F 0 "U?" H 4150 3600 50  0000 L CNN
+F 0 "U4" H 4150 3600 50  0000 L CNN
 F 1 "MCP2562-E/SN" H 4650 3600 50  0000 L CNN
 F 2 "Housings_SOIC:SOIC-8_3.9x4.9mm_Pitch1.27mm" H 4550 2750 50  0001 C CIN
@@
 $EndComp
 $Comp
-L +3.3V #PWR?
+L +3.3V #PWR070
 U 1 1 58D48987
 P 3200 3350
-F 0 "#PWR?" H 3200 3200 50  0001 C CNN
+F 0 "#PWR070" H 3200 3200 50  0001 C CNN
 F 1 "+3.3V" H 3200 3490 50  0000 C CNN
 F 2 "" H 3200 3350 50  0000 C CNN
@@
 $EndComp
 $Comp
-L C C?
+L C C36
 U 1 1 58D4898D
 P 3650 3550
-F 0 "C?" H 3675 3650 50  0000 L CNN
-F 1 "0.1uF" H 3675 3450 50  0000 L CNN
-F 2 "" H 3688 3400 50  0000 C CNN
+F 0 "C36" H 3675 3650 50  0000 L CNN
+F 1 "0.1u" H 3675 3450 50  0000 L CNN
+F 2 "Capacitors_SMD:C_0402" H 3688 3400 50  0001 C CNN
 F 3 "" H 3650 3550 50  0000 C CNN
+F 4 "CL05B104KO5NNNC" H 3650 3550 60  0001 C CNN "MPN"
 	1    3650 3550
 	1    0    0    -1
 $EndComp
 $Comp
-L GND #PWR?
+L GND #PWR071
 U 1 1 58D48994
 P 3650 3800
-F 0 "#PWR?" H 3650 3550 50  0001 C CNN
+F 0 "#PWR071" H 3650 3550 50  0001 C CNN
 F 1 "GND" H 3650 3650 50  0000 C CNN
 F 2 "" H 3650 3800 50  0000 C CNN
