File: power.sch (KiCad schematic (older format))
At the start: 49 parts

Commit message: stuff
Parts:
- added C38: 4.7u, Capacitors_SMD:C_1210, symbol C
- added JP4: Tie, Oddities:NetTie-I_Connected, symbol Jumper_NC_Small
- C16: renamed from C?; footprint (none) -> Capacitors_SMD:C_0402; MPN (none) -> GRM155R61A225KE95D
- C17: renamed from C?; footprint (none) -> Capacitors_SMD:C_0201; MPN (none) -> GRM033R71A682KA01D
- C18: renamed from C?; footprint (none) -> Capacitors_SMD:C_0805; MPN (none) -> CL21A475KAQNNNG
- C19: renamed from C?; footprint (none) -> Capacitors_SMD:C_0201; MPN (none) -> GRM0335C1H121JA01D
- C20: renamed from C?; footprint (none) -> Capacitors_SMD:C_0603; MPN (none) -> C0603C223K1RACTU
- C21: renamed from C?; value 10uF -> 10u; footprint Capacitors_SMD:C_0603 -> Capacitors_SMD:C_0805; MPN GRM188R61E105KA12D -> C0805C106K8PACTU
- C22: renamed from C?; footprint (none) -> Capacitors_SMD:C_0603; MPN (none) -> CC0603MRX5R7BB225
- C23: renamed from C?; value 22uF -> 22u; footprint Capacitors_SMD:C_0603 -> Capacitors_SMD:C_0805; MPN GRM188R61E105KA12D -> CL21A226KQCLRNC
- C24: renamed from C?; footprint (none) -> Capacitors_SMD:C_0805; MPN (none) -> CL21B104KCFNNNE
- C25: renamed from C?; footprint (none) -> Capacitors_SMD:C_1210; MPN (none) -> HMK325BJ475KM-PE
- C26, C27, C28: renamed from C?; footprint (none) -> Capacitors_SMD:C_0402; MPN (none) -> GRM155R61E104KA87D
- C29: renamed from C?; value 100n -> 0.1u; footprint (none) -> Capacitors_SMD:C_0805; MPN (none) -> CL21B104KCFNNNE
- C30: renamed from C?; value 10u -> 4.7u; footprint (none) -> Capacitors_SMD:C_1210; MPN (none) -> HMK325BJ475KM-PE
- C31: renamed from C?; footprint (none) -> Capacitors_SMD:C_1206; MPN (none) -> GRM31CR60J107ME39L
- C32: renamed from C?; footprint (none) -> Capacitors_SMD:C_0201; MPN (none) -> GRM033R71A222KA01D
- C33, C34, C35: renamed from C?; footprint (none) -> Capacitors_SMD:C_0201
- D3: renamed from D?; footprint (none) -> Diodes_SMD:D_SOD-123F; MPN (none) -> NRVTS260ESFT1G
- L1: renamed from L?; footprint (none) -> Inductors:Inductor_Taiyo-Yuden_NR-60xx; MPN (none) -> NR6045T220M
- Q1, Q2, Q3: renamed from Q?; footprint (none) -> hlib:SOT-1205
- R16, R17, R18, R19, R20, R21, R22, R25, R26, R32, R33: renamed from R?; footprint (none) -> Resistors_SMD:R_0201
- R23, R24, R28, R29, R30, R31: renamed from R?; footprint (none) -> Resistors_SMD:R_0402
- R27, R34: renamed from R?; footprint (none) -> hlib:R_shunt_4_terminal_2512
- U2: renamed from U?; footprint (none) -> TO_SOT_Packages_SMD:SOT-223; MPN (none) -> AZ1117CH-3.3TRG1
- U3: renamed from U?; footprint (none) -> crf1:TSSOP-56-PP
Connections:
- net GNDA is gone; now on net GND: C32.1, C33.1, C34.1, C35.1
- net DC_SUPPLY: now also C38.1
- net GND: now also C38.2, JP4.1; no longer Q2.1 (S), R27.1, R34.1
- net PHASE_B: now also Q2.5 (D), Q2.6 (D); no longer Q2.7 (D), Q2.8 (D)
- net PHASE_C: now also Q3.5 (D), Q3.6 (D); no longer Q3.7 (D), Q3.8 (D)
- net SL_A: now also Q1.3 (S), R27.4
- net SL_C: now also Q3.3 (S), R34.4
- net at R31.1: now also Q3.4 (G); no longer Q3.2 (G)
- net at R29.1: now also Q2.4 (G); no longer Q2.2 (G)
- net SL_B renamed GNDPWR
- net GNDPWR: now also Q2.3 (S), R27.1, R34.1, JP4.2
Other:
- moved on the sheet: C30

Commit message: stuff
Parts:
- JP4: footprint Oddities:NetTie-I_Connected -> hlib:NetTie-I_Connected_SMD
- U2: value AZ1117CH-3.3TRG1 -> AZ1117C; footprint TO_SOT_Packages_SMD:SOT-223 -> TO_SOT_Packages_SMD:SOT89-3_Housing; MPN AZ1117CH-3.3TRG1 -> AZ1117CR-3.3TRG1
Connections:
- net DC_SUPPLY: now also Q1.5 (D), Q1.6 (D), Q2.5 (D), Q2.6 (D), Q3.5 (D), Q3.6 (D); no longer Q1.7 (D), Q1.8 (D), Q2.7 (D), Q2.8 (D), Q3.7 (D), Q3.8 (D)
- net GND: no longer C30.2
- net GNDPWR: now also C30.2, Q2.1 (S); no longer Q2.3 (S)
- net PHASE_A: now also Q1.3 (S), Q1.7 (D), Q1.8 (D); no longer Q1.1 (S), Q1.5 (D), Q1.6 (D)
- net PHASE_B: now also Q2.3 (S), Q2.7 (D), Q2.8 (D); no longer Q2.1 (S), Q2.5 (D), Q2.6 (D)
- net PHASE_C: now also Q3.3 (S), Q3.7 (D), Q3.8 (D); no longer Q3.1 (S), Q3.5 (D), Q3.6 (D)
- net SL_A: now also Q1.1 (S); no longer Q1.3 (S)
- net SL_C: now also Q3.1 (S); no longer Q3.3 (S)
- net at Q1.2 (G): now also R24.1; no longer R23.1
- net at Q1.4 (G): now also R23.1; no longer R24.1
- net at Q3.2 (G): now also R31.1; no longer R30.1
- net at Q3.4 (G): now also R30.1; no longer R31.1
- net at Q2.2 (G): now also R29.1; no longer R28.1
- net at Q2.4 (G): now also R28.1; no longer R29.1
Other:
- note added: "The ground tie point on the \npcb is very close to where C30\nis located. And layout is easier \nthis way."
- moved on the sheet: Q1A, Q1B, Q2A, Q2B, Q3A, Q3B
Changed lines of the file:
@@
 P 2500 6300
 F 0 "U2" H 2500 6700 60  0000 C CNN
-F 1 "AZ1117CH-3.3TRG1" H 2950 6250 60  0000 C CNN
-F 2 "TO_SOT_Packages_SMD:SOT-223" H 2500 6200 60  0001 C CNN
+F 1 "AZ1117C" H 2950 6250 60  0000 C CNN
+F 2 "TO_SOT_Packages_SMD:SOT89-3_Housing" H 2500 6200 60  0001 C CNN
 F 3 "" H 2500 6200 60  0001 C CNN
-F 4 "AZ1117CH-3.3TRG1" H 2500 6300 60  0001 C CNN "MPN"
+F 4 "AZ1117CR-3.3TRG1" H 2500 6300 60  0001 C CNN "MPN"
 	1    2500 6300
 	1    0    0    -1
@@
 L BUK7K13-60E Q1
 U 1 1 59613EDB
+P 6950 2150
+F 0 "Q1" H 7150 2200 50  0000 L CNN
+F 1 "BUK7K13-60E" H 7150 2100 50  0000 L CNN
+F 2 "hlib:SOT-1205" H 7150 2250 50  0001 C CNN
+F 3 "" H 6950 2150 50  0001 C CNN
+	1    6950 2150
+	1    0    0    -1
+$EndComp
+$Comp
+L BUK7K13-60E Q1
+U 2 1 59613F4D
 P 6950 1350
 F 0 "Q1" H 7150 1400 50  0000 L CNN
@@
 F 2 "hlib:SOT-1205" H 7150 1450 50  0001 C CNN
 F 3 "" H 6950 1350 50  0001 C CNN
-	1    6950 1350
-	1    0    0    -1
-$EndComp
-$Comp
-L BUK7K13-60E Q1
-U 2 1 59613F4D
-P 6950 2150
-F 0 "Q1" H 7150 2200 50  0000 L CNN
-F 1 "BUK7K13-60E" H 7150 2100 50  0000 L CNN
-F 2 "hlib:SOT-1205" H 7150 2250 50  0001 C CNN
-F 3 "" H 6950 2150 50  0001 C CNN
-	2    6950 2150
+	2    6950 1350
 	1    0    0    -1
 $EndComp
@@
 F 4 "HMK325BJ475KM-PE" H 4650 1200 60  0001 C CNN "MPN"
 	1    4650 1200
-	1    0    0    -1
-$EndComp
-$Comp
-L GND #PWR042
-U 1 1 5962AD81
-P 4650 1350
-F 0 "#PWR042" H 4650 1100 50  0001 C CNN
-F 1 "GND" H 4650 1200 50  0000 C CNN
-F 2 "" H 4650 1350 50  0001 C CNN
-F 3 "" H 4650 1350 50  0001 C CNN
-	1    4650 1350
 	1    0    0    -1
 $EndComp
@@
 L BUK7K13-60E Q3
 U 1 1 596AEE48
+P 10400 2150
+F 0 "Q3" H 10600 2200 50  0000 L CNN
+F 1 "BUK7K13-60E" H 10600 2100 50  0000 L CNN
+F 2 "hlib:SOT-1205" H 10600 2250 50  0001 C CNN
+F 3 "" H 10400 2150 50  0001 C CNN
+	1    10400 2150
+	1    0    0    -1
+$EndComp
+$Comp
+L BUK7K13-60E Q3
+U 2 1 596AEE4E
 P 10400 1350
 F 0 "Q3" H 10600 1400 50  0000 L CNN
@@
 F 2 "hlib:SOT-1205" H 10600 1450 50  0001 C CNN
 F 3 "" H 10400 1350 50  0001 C CNN
-	1    10400 1350
-	1    0    0    -1
-$EndComp
-$Comp
-L BUK7K13-60E Q3
-U 2 1 596AEE4E
-P 10400 2150
-F 0 "Q3" H 10600 2200 50  0000 L CNN
-F 1 "BUK7K13-60E" H 10600 2100 50  0000 L CNN
-F 2 "hlib:SOT-1205" H 10600 2250 50  0001 C CNN
-F 3 "" H 10400 2150 50  0001 C CNN
-	2    10400 2150
+	2    10400 1350
 	1    0    0    -1
 $EndComp
@@
 L BUK7K13-60E Q2
 U 1 1 596AFA66
+P 8450 3750
+F 0 "Q2" H 8650 3800 50  0000 L CNN
+F 1 "BUK7K13-60E" H 8650 3700 50  0000 L CNN
+F 2 "hlib:SOT-1205" H 8650 3850 50  0001 C CNN
+F 3 "" H 8450 3750 50  0001 C CNN
+	1    8450 3750
+	1    0    0    -1
+$EndComp
+$Comp
+L BUK7K13-60E Q2
+U 2 1 596AFA6C
 P 8450 2950
 F 0 "Q2" H 8650 3000 50  0000 L CNN
@@
 F 2 "hlib:SOT-1205" H 8650 3050 50  0001 C CNN
 F 3 "" H 8450 2950 50  0001 C CNN
-	1    8450 2950
-	1    0    0    -1
-$EndComp
-$Comp
-L BUK7K13-60E Q2
-U 2 1 596AFA6C
-P 8450 3750
-F 0 "Q2" H 8650 3800 50  0000 L CNN
-F 1 "BUK7K13-60E" H 8650 3700 50  0000 L CNN
-F 2 "hlib:SOT-1205" H 8650 3850 50  0001 C CNN
-F 3 "" H 8450 3750 50  0001 C CNN
-	2    8450 3750
+	2    8450 2950
 	1    0    0    -1
 $EndComp
@@
 F 0 "JP4" H 6900 5630 50  0000 C CNN
 F 1 "Tie" H 6910 5490 50  0000 C CNN
-F 2 "Oddities:NetTie-I_Connected" H 6900 5550 50  0001 C CNN
+F 2 "hlib:NetTie-I_Connected_SMD" H 6900 5550 50  0001 C CNN
 F 3 "" H 6900 5550 50  0001 C CNN
 	1    6900 5550
@@
 	7100 5450 7100 5550
 Connection ~ 7100 5550
+$Comp
+L GNDPWR #PWR?
+U 1 1 59877EF7
+P 4650 1350
+F 0 "#PWR?" H 4650 1150 50  0001 C CNN
+F 1 "GNDPWR" H 4650 1220 50  0000 C CNN
+F 2 "" H 4650 1300 50  0001 C CNN
+F 3 "" H 4650 1300 50  0001 C CNN
+	1    4650 1350
+	1    0    0    -1
+$EndComp
+Text Notes 4900 1400 0    39   ~ 0
+The ground tie point on the \npcb is very close to where C30\nis located. And layout is easier \nthis way.
 $EndSCHEMATC
