File: small-bldc-hw.sch (KiCad schematic (older format))
At the start: 46 parts

Commit message: stuff
Parts:
- removed X?: 16 MHz, Crystals:Crystal_HC49-SD_SMD, symbol Crystal
- added J8, J9: CONN_01X01, Wire_Pads:SolderWirePad_single_SMD_5x10mm, symbol CONN_01X01
- added Y1: 16MHz, Crystals:Crystal_SMD_3225-4pin_3.2x2.5mm, symbol Crystal_GND24
- C1, C5: renamed from C?; value 18pF -> 10p; footprint Capacitors_SMD:C_0603 -> Capacitors_SMD:C_0201; MPN CL10C180JB8NNNC -> GRM0335C1H100JA01D
- C10: renamed from C?; value 10nF -> 10n; footprint Capacitors_SMD:C_0603 -> Capacitors_SMD:C_0402
- C11: renamed from C?; value 1uF -> 1u; footprint Capacitors_SMD:C_0603 -> Capacitors_SMD:C_0402
- C12, C14: renamed from C?; value 0.1uF -> 0.1u; footprint Capacitors_SMD:C_0603 -> Capacitors_SMD:C_0402; MPN GRM188R71C104KA01D -> CL05B104KO5NNNC
- C13, C8: renamed from C?; value 4.7uF -> 4.7u
- C15: renamed from C?; value 4n7 -> 4.7n; footprint (none) -> Capacitors_SMD:C_0201; MPN (none) -> GRM033R71A472KA01D
- C2: renamed from C?; value 0.1uF -> 0.1u; footprint Capacitors_SMD:C_0603 -> Capacitors_SMD:C_0402; MPN GRM188R71C104KA01D -> CL05A104KP5NNNC
- C3, C6, C7: renamed from C?; value 0.1uF -> 0.1u; footprint Capacitors_SMD:C_0603 -> Capacitors_SMD:C_0402
- C4: renamed from C?; value 4.7uF -> 4.7u; MPN GRM188R60J475KE19D -> CL10B475KQ8NQNC
- C9: renamed from C?; value 100n -> 0.1u; footprint (none) -> Capacitors_SMD:C_0402; MPN (none) -> CL05A104KP5NNNC
- D1, D2: renamed from D?; footprint SMD_Packages:SMD-0603 -> LEDs:LED_0603
- J1: renamed from J?; footprint (none) -> Connectors_JST:JST_SH_SM12B-SRSS-TB_12x1.00mm_Angled
- J2: renamed from J?; footprint (none) -> Connectors_JST:JST_SH_SM02B-SRSS-TB_02x1.00mm_Angled
- J3, J4, J5: renamed from J?; footprint (none) -> Wire_Pads:SolderWirePad_single_SMD_5x10mm
- J6, J7: renamed from J?; footprint (none) -> Connectors_JST:JST_SH_SM04B-SRSS-TB_04x1.00mm_Angled
- JP2, JP3: renamed from JP?; footprint (none) -> Resistors_SMD:R_0402
- P1: renamed from P?; footprint (none) -> Resistors_SMD:R_0402
- P2: renamed from P?; footprint Pin_Headers:Pin_Header_Straight_1x05 -> Connectors_JST:JST_SH_SM05B-SRSS-TB_05x1.00mm_Angled
- R1, R10, R11, R12: renamed from R?; footprint (none) -> Resistors_SMD:R_0603
- R13, R14, R15, R2, R9: renamed from R?; footprint (none) -> Resistors_SMD:R_0201
- R3, R4, R5, R6: renamed from R?; footprint SMD_Packages:SMD-0603 -> Resistors_SMD:R_0201
- R7, R8: renamed from R?; footprint (none) -> Resistors_SMD:R_0402
- gave numbers to parts that had none: 2
Connections:
- net labels added: GNDPWR
- wire segments 259 -> 221
Other:
- moved on the sheet: U1

Commit message: stuff
Parts:
- removed P1: CONN_02X01, Resistors_SMD:R_0402, symbol CONN_02X01
- J3, J4, J5: footprint Wire_Pads:SolderWirePad_single_SMD_5x10mm -> hlib:SolderWirePad_single_SMD_5x3.5mm
- J8, J9: footprint Wire_Pads:SolderWirePad_single_SMD_5x10mm -> hlib:SolderWirePad_single_SMD_5x3.5mm_holes
- JP1: footprint Pin_Headers:Pin_Header_Straight_1x02 -> Resistors_SMD:R_0603_HandSoldering
- Y1: footprint Crystals:Crystal_SMD_3225-4pin_3.2x2.5mm -> hlib:Crystal_SMD_3225-4pin_3.2x2.5mm
Connections:
- net CANH: now also R4.2
Changed lines of the file:
@@
-$EndComp
-$Comp
-L CONN_02X01 P1
-U 1 1 58D4CE36
-P 2750 6700
-F 0 "P1" H 2750 6800 50  0000 C CNN
-F 1 "CONN_02X01" H 2750 6600 50  0000 C CNN
-F 2 "Resistors_SMD:R_0402" H 2750 5500 50  0001 C CNN
-F 3 "" H 2750 5500 50  0000 C CNN
-	1    2750 6700
-	0    -1   -1   0
 $EndComp
 $Comp
@@
 F 0 "JP1" H 1700 2800 50  0000 C CNN
 F 1 "Boot Mode" H 1700 2700 50  0000 C CNN
-F 2 "Pin_Headers:Pin_Header_Straight_1x02" H 1700 1700 60  0001 C CNN
+F 2 "Resistors_SMD:R_0603_HandSoldering" H 1700 1700 60  0001 C CNN
 F 3 "" H 1700 1700 60  0000 C CNN
 	1    1700 2900
@@
 F 0 "J4" H 10450 4600 50  0000 C CNN
 F 1 "CONN_01X01" V 10550 4500 50  0001 C CNN
-F 2 "Wire_Pads:SolderWirePad_single_SMD_5x10mm" H 10450 4500 50  0001 C CNN
+F 2 "hlib:SolderWirePad_single_SMD_5x3.5mm" H 10450 4500 50  0001 C CNN
 F 3 "" H 10450 4500 50  0001 C CNN
 	1    10450 4500
@@
 F 0 "J3" H 10450 4100 50  0000 C CNN
 F 1 "CONN_01X01" V 10550 4000 50  0001 C CNN
-F 2 "Wire_Pads:SolderWirePad_single_SMD_5x10mm" H 10450 4000 50  0001 C CNN
+F 2 "hlib:SolderWirePad_single_SMD_5x3.5mm" H 10450 4000 50  0001 C CNN
 F 3 "" H 10450 4000 50  0001 C CNN
 	1    10450 4000
@@
 F 0 "J5" H 10450 5100 50  0000 C CNN
 F 1 "CONN_01X01" V 10550 5000 50  0001 C CNN
-F 2 "Wire_Pads:SolderWirePad_single_SMD_5x10mm" H 10450 5000 50  0001 C CNN
+F 2 "hlib:SolderWirePad_single_SMD_5x3.5mm" H 10450 5000 50  0001 C CNN
 F 3 "" H 10450 5000 50  0001 C CNN
 	1    10450 5000
@@
 $EndComp
 Wire Wire Line
-	2750 7000 2750 6950
-Wire Wire Line
 	1950 6650 2300 6650
 Wire Wire Line
@@
 	2350 7400 3100 7400
 Wire Wire Line
-	2750 6450 2750 6300
+	2750 7000 2750 6300
 Connection ~ 2750 6300
 Wire Wire Line
@@
 F 0 "J8" H 5600 6800 50  0000 C CNN
 F 1 "CONN_01X01" V 5700 6700 50  0000 C CNN
-F 2 "Wire_Pads:SolderWirePad_single_SMD_5x10mm" H 5600 6700 50  0001 C CNN
+F 2 "hlib:SolderWirePad_single_SMD_5x3.5mm_holes" H 5600 6700 50  0001 C CNN
 F 3 "" H 5600 6700 50  0001 C CNN
 	1    5600 6700
@@
 $EndComp
 Wire Wire Line
-	5400 6700 5200 6700
+	5200 6700 5400 6700
 $Comp
 L CONN_01X01 J9
@@
 F 0 "J9" H 5600 7150 50  0000 C CNN
 F 1 "CONN_01X01" V 5700 7050 50  0000 C CNN
-F 2 "Wire_Pads:SolderWirePad_single_SMD_5x10mm" H 5600 7050 50  0001 C CNN
+F 2 "hlib:SolderWirePad_single_SMD_5x3.5mm_holes" H 5600 7050 50  0001 C CNN
 F 3 "" H 5600 7050 50  0001 C CNN
 	1    5600 7050
@@
 F 0 "Y1" H 1025 3250 50  0000 L CNN
 F 1 "16MHz" H 1025 3175 50  0000 L CNN
-F 2 "Crystals:Crystal_SMD_3225-4pin_3.2x2.5mm" H 900 3050 50  0001 C CNN
+F 2 "hlib:Crystal_SMD_3225-4pin_3.2x2.5mm" H 900 3050 50  0001 C CNN
 F 3 "" H 900 3050 50  0001 C CNN
 F 4 "FA-238 16.0000MB-K3" H 900 3050 60  0001 C CNN "MPN"

Commit message: BOM stuff
Parts:
- J3, J4, J5: footprint hlib:SolderWirePad_single_SMD_5x3.5mm -> hlib:SolderWirePad_single_SMD_5x3.5mm_holes
Changed lines of the file:
@@
 F 0 "J4" H 10450 4600 50  0000 C CNN
 F 1 "CONN_01X01" V 10550 4500 50  0001 C CNN
-F 2 "hlib:SolderWirePad_single_SMD_5x3.5mm" H 10450 4500 50  0001 C CNN
+F 2 "hlib:SolderWirePad_single_SMD_5x3.5mm_holes" H 10450 4500 50  0001 C CNN
 F 3 "" H 10450 4500 50  0001 C CNN
 	1    10450 4500
@@
 F 0 "J3" H 10450 4100 50  0000 C CNN
 F 1 "CONN_01X01" V 10550 4000 50  0001 C CNN
-F 2 "hlib:SolderWirePad_single_SMD_5x3.5mm" H 10450 4000 50  0001 C CNN
+F 2 "hlib:SolderWirePad_single_SMD_5x3.5mm_holes" H 10450 4000 50  0001 C CNN
 F 3 "" H 10450 4000 50  0001 C CNN
 	1    10450 4000
@@
 F 0 "J5" H 10450 5100 50  0000 C CNN
 F 1 "CONN_01X01" V 10550 5000 50  0001 C CNN
-F 2 "hlib:SolderWirePad_single_SMD_5x3.5mm" H 10450 5000 50  0001 C CNN
+F 2 "hlib:SolderWirePad_single_SMD_5x3.5mm_holes" H 10450 5000 50  0001 C CNN
 F 3 "" H 10450 5000 50  0001 C CNN
 	1    10450 5000
