File: small-bldc-hw.kicad_pcb (KiCad board)
At the start: 4 copper layers, 65 x 22.4 mm, 98 parts, among them J1 More IO, J2 TEMP, J3 CONN_01X01, J4 CONN_01X01, J5 CONN_01X01, J6 CAN, J7 I2C, J8 CONN_01X01, J9 CONN_01X01, P2 SWD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

Commit message: labelled the pads
Other:
- board text added: "A"
- board text added: "B"
- board text added: "C"
- board text added: "DC_IN"
- board text added: "GND"
- board text added: "onwyd 1"
Changed lines of the file:
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@@
     (area 118.26896 88.33446 185.900001 113.67752)
     (thickness 1.6)
-    (drawings 4)
+    (drawings 10)
     (tracks 3486)
     (zones 0)
@@
   (layers
     (0 F.Cu signal)
-    (1 In1.Cu signal)
-    (2 In2.Cu signal)
-    (31 B.Cu signal)
+    (1 In1.Cu signal hide)
+    (2 In2.Cu signal hide)
+    (31 B.Cu signal hide)
     (35 F.Paste user)
     (36 B.SilkS user)
@@
     (visible_elements FFFFEF7F)
     (pcbplotparams
-      (layerselection 0x00008_00000000)
-      (usegerberextensions false)
+      (layerselection 0x010a0_80000007)
+      (usegerberextensions true)
       (excludeedgelayer true)
       (linewidth 0.100000)
@@
       (drillshape 0)
       (scaleselection 1)
-      (outputdirectory ""))
+      (outputdirectory gerbers/))
   )
   (net 0 "")
@@
     (tags "MesurementPoint Square SMDPad 5mmx10mm ")
     (attr smd)
-    (fp_text reference J5 (at 1.1 -2.1) (layer F.SilkS)
+    (fp_text reference J5 (at 1.1 -2.1) (layer F.SilkS) hide
       (effects (font (size 0.3048 0.3048) (thickness 0.0762)))
     )
@@
     (tags "MesurementPoint Square SMDPad 5mmx10mm ")
     (attr smd)
-    (fp_text reference J4 (at 1.15 -2.05) (layer F.SilkS)
+    (fp_text reference J4 (at 1.15 -2.05) (layer F.SilkS) hide
       (effects (font (size 0.3048 0.3048) (thickness 0.0762)))
     )
@@
     (tags "MesurementPoint Square SMDPad 5mmx10mm ")
     (attr smd)
-    (fp_text reference J3 (at -0.741 2.1155) (layer F.SilkS)
+    (fp_text reference J3 (at -0.741 2.1155) (layer F.SilkS) hide
       (effects (font (size 0.3048 0.3048) (thickness 0.0762)))
     )
@@
     (tags "MesurementPoint Square SMDPad 5mmx10mm ")
     (attr smd)
-    (fp_text reference J8 (at 0.95 -2.15) (layer F.SilkS)
+    (fp_text reference J8 (at 0.95 -2.15) (layer F.SilkS) hide
       (effects (font (size 0.3048 0.3048) (thickness 0.0762)))
     )
@@
     (tags "MesurementPoint Square SMDPad 5mmx10mm ")
     (attr smd)
-    (fp_text reference J9 (at 2.931 1.7153 180) (layer F.SilkS)
+    (fp_text reference J9 (at 2.931 1.7153 180) (layer F.SilkS) hide
       (effects (font (size 0.3048 0.3048) (thickness 0.0762)))
     )
@@
   (module hlib:SOT-1205_open_vias (layer F.Cu)
     (at 174.258 97.2346)
-    (fp_text reference Q1 (at 4.542 2.3154 270) (layer F.SilkS)
+    (fp_text reference Q1 (at -3.608 0.3654 270) (layer F.SilkS)
       (effects (font (size 0.5 0.5) (thickness 0.125)))
     )
@@
   (module hlib:SOT-1205_open_vias (layer F.Cu)
     (at 174.258 103.205)
-    (fp_text reference Q2 (at 4.542 2.345 270) (layer F.SilkS)
+    (fp_text reference Q2 (at -3.558 -1.955 270) (layer F.SilkS)
       (effects (font (size 0.5 0.5) (thickness 0.125)))
     )
@@
   (module hlib:SOT-1205_open_vias (layer F.Cu)
     (at 174.258 109.175)
-    (fp_text reference Q3 (at 4.542 2.125 270) (layer F.SilkS)
+    (fp_text reference Q3 (at -3.608 -1.525 270) (layer F.SilkS)
       (effects (font (size 0.5 0.5) (thickness 0.125)))
     )
@@
     )
   )
+  (gr_text GND (at 166.9 91.5 90) (layer F.SilkS)
+    (effects (font (size 0.8 0.8) (thickness 0.14)))
+  )
+  (gr_text A (at 179.95 94.35) (layer F.SilkS)
+    (effects (font (size 0.8 0.8) (thickness 0.14)))
+  )
+  (gr_text B (at 183.3 95.1) (layer F.SilkS)
+    (effects (font (size 0.8 0.8) (thickness 0.14)))
+  )
+  (gr_text C (at 183.8 101.3) (layer F.SilkS)
+    (effects (font (size 0.8 0.8) (thickness 0.14)))
+  )
+  (gr_text DC_IN (at 181.8 107.4) (layer F.SilkS)
+    (effects (font (size 0.8 0.8) (thickness 0.14)))
+  )
+  (gr_text "onwyd 1" (at 122.75 98.35) (layer F.SilkS)
+    (effects (font (size 0.8 0.8) (thickness 0.11)))
+  )
   (gr_line (start 119.888 112.0775) (end 119.888 89.7255) (layer Edge.Cuts) (width 0.1))

Commit message: idk
Other:
- net class Default: clearance 0.1524 -> 0.153924
- net class smallpower: clearance 0.1524 -> 0.153924
- rule trace_clearance: 0.1524 -> 0.153924
Changed lines of the file:
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@@
   (page A4)
   (layers
-    (0 F.Cu signal)
-    (1 In1.Cu signal hide)
+    (0 F.Cu signal hide)
+    (1 In1.Cu signal)
     (2 In2.Cu signal hide)
-    (31 B.Cu signal hide)
+    (31 B.Cu signal)
     (35 F.Paste user)
     (36 B.SilkS user)
@@
   (setup
     (last_trace_width 0.1524)
-    (trace_clearance 0.1524)
+    (trace_clearance 0.153924)
     (zone_clearance 0.508)
     (zone_45_only no)
@@
   (net 89 /CAN_TX)
   (net_class Default "This is the default net class."
-    (clearance 0.1524)
+    (clearance 0.153924)
     (trace_width 0.1524)
     (via_dia 0.6858)
@@
   )
   (net_class smallpower ""
-    (clearance 0.1524)
+    (clearance 0.153924)
     (trace_width 0.4572)
     (via_dia 0.6858)
@@
       (pts
         (xy 184.9 89.75) (xy 178.8 89.55) (xy 178.9 93.85) (xy 173.7 94.4) (xy 172.2 94.5)
-        (xy 172.95 99.5) (xy 177.6 99.5) (xy 178.45 95.4) (xy 184.9 95.4)
+        (xy 172.95 99.5) (xy 177.7 97.75) (xy 178.85 96.3) (xy 184.9 95.4)
       )
     )
@@
     (polygon
       (pts
-        (xy 184.9 95.4) (xy 178.45 95.4) (xy 177.6 99.6) (xy 172.6 99.65) (xy 172.6 106.55)
-        (xy 178.25 105.1) (xy 179.05 101.4) (xy 184.85 101.5) (xy 184.9 95.45)
+        (xy 184.9 95.4) (xy 178.45 95.4) (xy 176.1 98.4) (xy 172.6 99.65) (xy 172.6 106.55)
+        (xy 177.95 104.2) (xy 179.05 101.4) (xy 184.85 101.5) (xy 184.9 95.45)
       )
     )
@@
       (pts
         (xy 171.15 106.05) (xy 171.15 112.05) (xy 184.8 112.05) (xy 184.85 101.5) (xy 179.05 101.4)
-        (xy 178.25 105.1)
+        (xy 177 103.1)
       )
     )

Commit message: I think something relating to planes was changed
Routing:
- net GNDPWR: track 72.2 -> 72.5 mm, vias 4 -> 5
Other:
- net class Default: clearance 0.153924 -> 0.1524
- net class smallpower: clearance 0.153924 -> 0.1524
- rule trace_clearance: 0.153924 -> 0.1524
